Commit message: updated the code for pub sub nodes of sensor need to look into lidar and camera publishers eal time working

File: install/my_robot/share/my_robot/description/robot.urdf.xacro (robot description, xacro)
@@ -3,3 +3,4 @@
     <xacro:include filename="robot_core.xacro" />
     <xacro:include filename="gazebo_controller.xacro" />
+    <xacro:include filename="sensors.xacro" />
 </robot>

File: install/my_robot/share/my_robot/description/robot_core.xacro (robot description, xacro)
@@ -179,102 +179,3 @@
         <material>Gazebo/Blue</material>
     </gazebo>
-    <!-- Sensors -->
-    <!-- LiDAR Sensor -->
-    <!-- Define the LiDAR -->
-    <xacro:property name="lidar_beam_count" value="360"/> <!-- The number of laser beams emitted by the LiDAR, set to 360 in this case. -->
-    <xacro:property name="lidar_fov" value="1.57"/> <!-- Approximately 90 degrees in radians pi/2 -->
-    <xacro:property name="lidar_range" value="30.0"/> <!-- Maximum range in meters -->
-    <link name="lidar_link">
-        <visual>
-            <origin xyz="0 0 0" rpy="0 0 0"/>
-            <geometry>
-                <cylinder length="0.05" radius="0.03"/>
-            </geometry>
-            <material name="red"/>
-        </visual>
-        <collision>
-            <origin xyz="0 0 0" rpy="0 0 0"/>
-            <geometry>
-                <cylinder length="0.05" radius="0.06"/>
-            </geometry>
-        </collision>
-        <xacro:inertial_cylinder mass="0.1" length="0.05" radius="0.06">
-            <origin xyz="0 0 0" rpy="0 0 0"/>
-        </xacro:inertial_cylinder>
-    </link>
-    <joint name="lidar_joint" type="continuous">
-        <parent link="smaller_box"/>
-        <child link="lidar_link"/>
-        <origin xyz="0 0 0.07" rpy="0 0 0"/>
-        <axis xyz="0 0 1"/>
-    </joint>
-    <gazebo reference="lidar_link">
-        <material>Gazebo/Red</material>
-    </gazebo>
-    <gazebo reference="lidar_link">
-        <sensor type="lidar" name="lidar_link_sensor">
-          <pose>0 0 0 0 0 0</pose>
-          <visualize>false</visualize>
-          <update_rate>10.0</update_rate>
-          <ray>
-            <scan>
-              <horizontal>
-                <samples>${lidar_beam_count}</samples>
-                <min_angle>-${lidar_fov/2}</min_angle>
-                <max_angle>${lidar_fov/2}</max_angle>
-              </horizontal>
-            </scan>
-            <range>
-              <min>0.02</min>
-              <max>${lidar_range}</max>
-            </range>
-          </ray>
-        </sensor>
-    </gazebo>
-    <!-- Camera -->
-    <!-- Define the camera properties -->
-    <xacro:property name="camera_fov" value="1.047"/> <!-- Approximately 60 degrees in radians -->
-    <xacro:property name="camera_width" value="640"/>
-    <xacro:property name="camera_height" value="480"/>
-    <link name="camera_link">
-        <visual>
-            <origin xyz="0 0 0" rpy="0 0 0"/>
-            <geometry>
-                <box size="0.05 0.15 0.05"/>
-            </geometry>
-            <material name="red"/>
-        </visual>
-        <collision>
-            <origin xyz="0 0 0" rpy="0 0 0"/>
-            <geometry>
-              <box size= "0.05 0.15 0.05"/>
-            </geometry>
-        </collision>
-    </link>
-    <joint name="camera_joint" type="fixed">
-        <parent link="chassis"/>
-        <child link="camera_link"/>
-        <origin xyz="0.42 0 0.025" rpy="0 0 0"/>
-    </joint>
-    <gazebo reference="camera_link">
-        <material>Gazebo/Red</material>
-    </gazebo>
-    <gazebo reference="camera_link">
-        <sensor type="camera" name="camera_link_sensor">
-          <pose>0 0 0 0 0 0</pose>
-          <visualize>false</visualize>
-          <update_rate>30.0</update_rate>
-          <camera name="camera_link">
-            <horizontal_fov>${camera_fov}</horizontal_fov>
-            <image>
-              <width>${camera_width}</width>
-              <height>${camera_height}</height>
-            </image>
-            <clip>
-              <near>0.01</near>
-              <far>100</far>
-            </clip>
-          </camera>
-        </sensor>
-    </gazebo>
 </robot>
