Commit message: added mapping fileds

File: install/my_robot/share/my_robot/description/gazebo_controller.xacro (robot description, xacro)
@@ -3,11 +3,4 @@
     <gazebo>
         <plugin name='skid_steer_drive' filename='libgazebo_ros_diff_drive.so'>
-            <ros>
-              <!-- Set namespace -->
-              <namespace>/demo</namespace>
-              <!-- Remap default topics -->
-              <remapping>cmd_vel:=cmd_demo</remapping>
-              <remapping>odom:=odom_demo</remapping>
-            </ros>
             <!-- Update rate -->
             <update_rate>500</update_rate>
@@ -32,6 +25,6 @@
             <publish_odom_tf>true</publish_odom_tf>
             <publish_wheel_tf>true</publish_wheel_tf>
-            <odometry_frame>odom_demo</odometry_frame>
-            <robot_base_frame>chassis</robot_base_frame>
+            <odometry_frame>odom</odometry_frame>
+            <robot_base_frame>base_link</robot_base_frame>
         </plugin>
     </gazebo>

File: install/my_robot/share/my_robot/description/robot_core.xacro (robot description, xacro)
@@ -2,4 +2,5 @@
 <robot xmlns:xacro="http://www.ros.org/wiki/xacro" name="robot">
     <xacro:include filename="inertial_macros.xacro"/>
+    <!-- chasis color -->
     <material name="white">
         <color rgba="1 1 1 1" />
@@ -19,4 +20,12 @@
     <!-- BASE LINK -->
     <link name="base_link">
+    </link>
+    <!-- Base foot print link for slam application-->
+    <joint name="base_footprint_joint" type="fixed">
+        <parent link="base_link"/>
+        <child link="base_footprint"/>
+        <origin xyz="0 0 0"/>
+    </joint>
+    <link name="base_footprint">
     </link>
     <!-- CHASSIS LINK -->

File: install/my_robot/share/my_robot/description/sensors.xacro (robot description, xacro)
@@ -41,5 +41,5 @@
                 </range>
             </ray>
-            <plugin name="laser_controller" filename="gazelibbo_ros_ray_sensor.so">
+            <plugin name="laser_controller" filename="libgazebo_ros_ray_sensor.so">
                 <ros>
                     <argument>~/out:=scan</argument>
